Commit message: Measure drivetrain constants: 224 edges/wheel-rev, 60mm wheels
encoder.h derived EDGES_PER_WHEEL_REV from datasheet-typical constants
(ENCODER_CPR 11 * 4 * GEAR_RATIO 34 = 1496), both marked "may vary,
measure". Measured it directly instead by hand-turning the FR wheel
exactly 10 revolutions with the bridges disabled and reading the
counter: 2240 and 2244 over two runs — 224 edges/rev, the two runs
0.18% apart.

The old value was wrong by 6.7x, for two compounding reasons: the
gearbox is ~1:20 rather than 1:34 (224 / 11 = 20.4), and the firmware's
software EXTI decode counts channel A's rising edge only — 1x, not the
4x a hardware quadrature peripheral would give. Odometry scales
directly off this constant, so it would have misreported distance by
that same factor.

Measuring the end-to-end figure is what makes it right; it needs no
separate knowledge of CPR, gearing, or edge-counting scheme, and
inherently tracks whatever those really are. Kept as a measured
constant rather than a derived one for that reason.

Propagated to every consumer, which had each hardcoded the derived
value independently: the ROS 2 hardware interface and the protocol
simulator. Wheel radius corrected alongside it — the wheels are 60mm
diameter, not the 65mm assumed in the hardware interface, URDF and
controllers.yaml.

Also raises the SIL mock's max_wheel_rps from 0.18 to 5.0 rev/s. The
old figure (~11 RPM at the wheel) was not physical; it existed to make
counts visible under the inflated 1496 constant, and with a correct 224
it produced sub-one-edge accumulation, failing SIL's encoder assertion.
The new value is an order-of-magnitude estimate for a 1:20 JGA25-370 at
12V, not a measurement — SIL asserts control-path logic, never speed
accuracy. Real motor RPM is still unmeasured.

Adds encoder_count: a passive, motors-never-driven target used to take
the measurement, kept for re-measuring if the drivetrain changes.

File: ros2_ws/src/mcr_description/urdf/mcr.urdf.xacro (robot description, xacro)
@@ -21,5 +21,5 @@
   <!-- Parameters                                                    -->
   <!-- ============================================================ -->
-  <xacro:property name="wheel_radius"   value="0.0325"/>  <!-- m -->
+  <xacro:property name="wheel_radius"   value="0.030"/>   <!-- m (60mm mecanum wheels, measured) -->
   <xacro:property name="wheel_width"    value="0.026"/>   <!-- m -->
   <xacro:property name="wheel_mass"     value="0.05"/>    <!-- kg -->

Commit message: fix(kinematics): replace estimated lx/ly with measured values
lx=0.10/ly=0.12 had been estimates since M4, flagged in the roadmap as
never measured. Measured today with a tape measure: front-rear axle
center distance 0.125 m (lx=0.0625), left-right axle center distance
0.18 m (ly=0.09 -- derived from 21 cm outer-edge-to-outer-edge minus
one 3 cm wheel width, not two: each wheel's center sits half a wheel
width inboard of its own outer edge, so only one full wheel width
separates outer-edge span from axle-center span, not two half-widths
counted from each side as two separate wheel widths).

Updated all six locations the M4 roadmap note listed as needing to
stay in sync: firmware remote_control.c and its host test, the URDF,
the ROS 2 hardware interface default and its test, and controllers.yaml
(as the combined lx+ly sum that package's kinematics config expects).
wheel_radius (0.0325 in the two test fixtures) is untouched -- that's
the separate, already-flagged T5 question about whether the test value
is intentional or leftover, not part of this change.

firmware/Core/Test/test_mecanum_ik.c passes host-built after the
change (all five cases derive their expected values from the LX/LY
macros rather than hardcoding numbers, so they stay self-consistent).
ros2_ws/src/mcr_bringup/test/test_mecanum_kinematics.cpp is the same
shape (round-trip and sign-pattern checks) but wasn't run today --
would need a colcon build.

File: ros2_ws/src/mcr_description/urdf/mcr.urdf.xacro (robot description, xacro)
@@ -24,6 +24,6 @@
   <xacro:property name="wheel_width"    value="0.026"/>   <!-- m -->
   <xacro:property name="wheel_mass"     value="0.05"/>    <!-- kg -->
-  <xacro:property name="lx"             value="0.10"/>    <!-- half wheelbase (m) -->
-  <xacro:property name="ly"             value="0.12"/>    <!-- half track width (m) -->
+  <xacro:property name="lx"             value="0.0625"/> <!-- half wheelbase (m), measured 2026-08-30 -->
+  <xacro:property name="ly"             value="0.09"/>   <!-- half track width (m), measured 2026-08-30 -->
   <xacro:property name="base_length"    value="0.26"/>    <!-- chassis length -->
   <xacro:property name="base_width"     value="0.22"/>    <!-- chassis width -->
